File: reck-pcba.kicad_pcb (KiCad board)
At the start: 2 copper layers, 19 parts, among them J1 Conn_01x03_Pin, SW1 PTS810_SJM_250_SMTR_LFS, SW2 PTS810_SJM_250_SMTR_LFS, SW3 PTS810_SJM_250_SMTR_LFS, SW4 PTS810_SJM_250_SMTR_LFS, U1 ESP32-S3FN8, U10 USBLC6-2P6, U11 WS2812B, U12 SAM-M10Q-00B, U13 MCP4728, U14 SN74LVC1T45DBV, U15 TPS62912RPUR, U16 TPS62912RPUR, U2 SN74LVC1T45DBV, U3 DRV8231ADSGR, U6 ADS1015IDGS, U7 WS2812B, U8 WS2812B, U9 WS2812B

Commit message: Full Schematics Complete - Changed uC to ESP32-S3-WROOM-2 to allow for pinout discussion. - Moved buck regulators to main sheet. - Added titles and descriptions to each Sensor, Interface, or concept. - Added LCD. - Changed DAC to single-channel variant. - Added I2C Laser Time-of-Flight Sensor. - Added Environmental Sensor. - Updated pinout on uC.
Parts:
- removed J1: Conn_01x03_Pin, Connector_PinHeader_2.54mm:PinHeader_1x03_P2.54mm_Vertical
- removed SW1, SW2, SW3, SW4: PTS810_SJM_250_SMTR_LFS, reck-switches:PTS810_SJM_250_SMTR_LFS
- removed U1: ESP32-S3FN8, reck-ics:QFN-56-1EP_7x7mm_P0.4mm_EP4x4mm
- removed U10: USBLC6-2P6, Package_TO_SOT_SMD:SOT-666
- removed U11, U7, U8, U9: WS2812B, reck-ics:WS2812B
- removed U12: SAM-M10Q-00B, reck-ics:SAM-M10Q
- removed U13: MCP4728, Package_SO:MSOP-10_3x3mm_P0.5mm
- removed U14, U2: SN74LVC1T45DBV, Package_TO_SOT_SMD:SOT-23-6
- removed U15, U16: TPS62912RPUR, reck-ics:VQFN-HR-10_2x2mm
- removed U3: DRV8231ADSGR, Package_SON:WSON-8-1EP_2x2mm_P0.5mm_EP0.9x1.6mm
- removed U6: ADS1015IDGS, Package_SO:TSSOP-10_3x3mm_P0.5mm

Commit message: Added new uC, Power, and Motor support - Updated ESP32-C3 to ESP32-S3 due to GPIO constraints - Using two buck regulators for servo 5V power and board 3V3
Parts:
- added J1: Conn_01x03_Pin, Connector_PinHeader_2.54mm:PinHeader_1x03_P2.54mm_Vertical, F.Cu at (122.1, 83.9)
- added SW1: PTS810_SJM_250_SMTR_LFS, reck-switches:PTS810_SJM_250_SMTR_LFS, F.Cu at (116.4, 66.9)
- added SW2: PTS810_SJM_250_SMTR_LFS, reck-switches:PTS810_SJM_250_SMTR_LFS, F.Cu at (116.4, 71.7)
- added SW3: PTS810_SJM_250_SMTR_LFS, reck-switches:PTS810_SJM_250_SMTR_LFS, F.Cu at (116.4, 76.4)
- added SW4: PTS810_SJM_250_SMTR_LFS, reck-switches:PTS810_SJM_250_SMTR_LFS, F.Cu at (116.4, 81.2)
- added U1: ESP32-S3FN8, reck-ics:QFN-56-1EP_7x7mm_P0.4mm_EP4x4mm, F.Cu at (129.1, 86.2)
- added U10: USBLC6-2P6, Package_TO_SOT_SMD:SOT-666, F.Cu at (121.8, 93.1)
- added U11: WS2812B, reck-ics:WS2812B, F.Cu at (108.4, 86.0)
- added U12: SAM-M10Q-00B, reck-ics:SAM-M10Q, F.Cu at (128.8, 73.1)
- added U13: MCP4728, Package_SO:MSOP-10_3x3mm_P0.5mm, F.Cu at (108.5, 91.4)
- added U14: SN74LVC1T45DBV, Package_TO_SOT_SMD:SOT-23-6, F.Cu at (115.2, 90.6)
- added U15: TPS62912RPUR, reck-ics:VQFN-HR-10_2x2mm, F.Cu at (141.6, 66.2)
- added U16: TPS62912RPUR, reck-ics:VQFN-HR-10_2x2mm, F.Cu at (141.6, 69.6)
- added U2: SN74LVC1T45DBV, Package_TO_SOT_SMD:SOT-23-6, F.Cu at (115.2, 85.9)
- added U3: DRV8231ADSGR, Package_SON:WSON-8-1EP_2x2mm_P0.5mm_EP0.9x1.6mm, F.Cu at (133.6, 92.8)
- added U6: ADS1015IDGS, Package_SO:TSSOP-10_3x3mm_P0.5mm, F.Cu at (127.9, 93.2)
- added U7: WS2812B, reck-ics:WS2812B, F.Cu at (108.4, 67.6)
- added U8: WS2812B, reck-ics:WS2812B, F.Cu at (108.4, 73.7)
- added U9: WS2812B, reck-ics:WS2812B, F.Cu at (108.4, 79.9)
