File: reck-pcba.kicad_pcb (KiCad board)
At the start: 2 copper layers, 0 parts

Commit message: updated
Parts:
- added BZ1: CEM-1206S, reck-audio:CEM-1206S, F.Cu at (301.6, 96.1)
- added C1: 2.2nF, Capacitor_SMD:C_0603_1608Metric, F.Cu at (276.8, 77.5)
- added C10: 1uF, Capacitor_SMD:C_0603_1608Metric, F.Cu at (246.4, 145.0)
- added C10: 1uF, Capacitor_SMD:C_0603_1608Metric, F.Cu at (264.0, 145.0)
- added C11: 22uF, Capacitor_SMD:C_0805_2012Metric, F.Cu at (281.4, 120.9)
- added C12: 22uF, Capacitor_SMD:C_0805_2012Metric, F.Cu at (274.6, 146.4)
- added C12: 22uF, Capacitor_SMD:C_0805_2012Metric, F.Cu at (257.0, 146.4)
- added C13: 100nF, Capacitor_SMD:C_0603_1608Metric, F.Cu at (276.8, 92.6)
- added C14: 22uF, Capacitor_SMD:C_0805_2012Metric, F.Cu at (281.4, 126.9)
- added C15: 22uF, Capacitor_SMD:C_0805_2012Metric, F.Cu at (255.0, 146.4)
- added C15: 22uF, Capacitor_SMD:C_0805_2012Metric, F.Cu at (272.6, 146.4)
- added C16: 100nF, Capacitor_SMD:C_0603_1608Metric, F.Cu at (276.8, 95.1)
- added C17: 22uF, Capacitor_SMD:C_0805_2012Metric, F.Cu at (285.9, 120.9)
- added C18: 22uF, Capacitor_SMD:C_0805_2012Metric, F.Cu at (253.0, 146.4)
- added C18: 22uF, Capacitor_SMD:C_0805_2012Metric, F.Cu at (270.6, 146.4)
- added C19: 100nF, Capacitor_SMD:C_0603_1608Metric, F.Cu at (276.8, 97.6)
- added C2: 10uF, Capacitor_SMD:C_0805_2012Metric, F.Cu at (277.0, 120.9)
- added C20: 100nF, Capacitor_SMD:C_0603_1608Metric, F.Cu at (276.8, 100.1)
- added C21: 100nF, Capacitor_SMD:C_0603_1608Metric, F.Cu at (276.8, 102.6)
- added C22: 100nF, Capacitor_SMD:C_0603_1608Metric, F.Cu at (280.8, 77.5)
- added C23: 100nF, Capacitor_SMD:C_0603_1608Metric, F.Cu at (280.8, 80.0)
- added C24: 22uF, Capacitor_SMD:C_0805_2012Metric, F.Cu at (285.9, 126.9)
- added C25: 100nF, Capacitor_SMD:C_0603_1608Metric, F.Cu at (280.8, 82.5)
- added C26: 47uF, Capacitor_SMD:CP_Elec_6.3x5.9, F.Cu at (293.4, 123.4)
- added C27: 100nF, Capacitor_SMD:C_0603_1608Metric, F.Cu at (280.8, 85.1)
- added C28: 100nF, Capacitor_SMD:C_0603_1608Metric, F.Cu at (280.8, 87.6)
- added C29: 100nF, Capacitor_SMD:C_0603_1608Metric, F.Cu at (280.8, 90.1)
- added C3: 10uF, Capacitor_SMD:C_0805_2012Metric, F.Cu at (268.1, 141.8)
- added C3: 10uF, Capacitor_SMD:C_0805_2012Metric, F.Cu at (250.6, 141.8)
- added C30: 100nF, Capacitor_SMD:C_0603_1608Metric, F.Cu at (280.8, 92.6)
- added C31: 100nF, Capacitor_SMD:C_0603_1608Metric, F.Cu at (280.8, 95.1)
- added C32: 100nF, Capacitor_SMD:C_0603_1608Metric, F.Cu at (280.8, 97.6)
- added C33: 100nF, Capacitor_SMD:C_0603_1608Metric, F.Cu at (280.8, 100.1)
- added C34: 100nF, Capacitor_SMD:C_0603_1608Metric, F.Cu at (280.8, 102.6)
- added C35: 100nF, Capacitor_SMD:C_0603_1608Metric, F.Cu at (284.8, 77.5)
- added C36: 100nF, Capacitor_SMD:C_0603_1608Metric, F.Cu at (284.8, 80.0)
- added C37: 10uF, Capacitor_SMD:C_0805_2012Metric, F.Cu at (285.9, 129.9)
- added C4: 10uF, Capacitor_SMD:C_0805_2012Metric, F.Cu at (277.0, 126.9)
- added C5: 10uF, Capacitor_SMD:C_0805_2012Metric, F.Cu at (268.1, 139.8)
- added C5: 10uF, Capacitor_SMD:C_0805_2012Metric, F.Cu at (250.6, 139.8)
- added C6: 1uF, Capacitor_SMD:C_0603_1608Metric, F.Cu at (276.8, 80.0)
- added C7: 2.2nF, Capacitor_SMD:C_0603_1608Metric, F.Cu at (276.8, 82.5)
- added C8: 1uF, Capacitor_SMD:C_0603_1608Metric, F.Cu at (276.8, 85.1)
- added C9: 2.2nF, Capacitor_SMD:C_0603_1608Metric, F.Cu at (250.4, 143.6)
- added C9: 2.2nF, Capacitor_SMD:C_0603_1608Metric, F.Cu at (268.0, 143.6)
- added D1: LED, LED_SMD:LED_0603_1608Metric, F.Cu at (267.5, 120.1)
- added D2: CDBA340L-HF, Diode_SMD:D_SMA, F.Cu at (310.8, 59.3)
- added D3: LED, LED_SMD:LED_0603_1608Metric, F.Cu at (267.5, 122.7)
- added D4: CDBA340L-HF, Diode_SMD:D_SMA, F.Cu at (310.8, 63.8)
- added D5: 1SMA5928BT3G, Diode_SMD:D_SMA, F.Cu at (310.8, 68.4)
- added D6: LED, LED_SMD:LED_0603_1608Metric, F.Cu at (267.5, 125.3)
- added D7: LED, LED_SMD:LED_0603_1608Metric, F.Cu at (267.5, 127.9)
- added D8: LED, LED_SMD:LED_0603_1608Metric, F.Cu at (267.5, 130.5)
- added D9: CDBA340L-HF, Diode_SMD:D_SMA, F.Cu at (310.8, 72.9)
- added J1: USB4105-GF-A, Connector_USB:USB_C_Receptacle_GCT_USB4105-xx-A_16P_TopMnt_Horizontal, F.Cu at (251.6, 126.2)
- added J2: 575-4, reck-connectors:575-4, F.Cu at (311.5, 42.8)
- added J3: 575-4, reck-connectors:575-4, F.Cu at (311.5, 52.3)
- added J4: Conn_01x03_Pin, Connector_PinHeader_2.54mm:PinHeader_1x03_P2.54mm_Vertical, F.Cu at (258.5, 121.1)
- added J5: Conn_01x03_Pin, Connector_PinHeader_2.54mm:PinHeader_1x03_P2.54mm_Vertical, F.Cu at (263.2, 121.1)
- added J6: TBL002A-350-02GR-2OR, reck-connectors:TBL002A-350-02GR-2OR, F.Cu at (229.7, 121.9)
- added L1: 2.2uH, Inductor_SMD:L_1210_3225Metric, F.Cu at (311.2, 106.0)
- added L1: 2.2uH, Inductor_SMD:L_1210_3225Metric, F.Cu at (251.6, 150.2)
- added L2: 2.2uH, Inductor_SMD:L_1210_3225Metric, F.Cu at (269.2, 150.2)
- added Q1: BC846, Package_TO_SOT_SMD:SOT-23, F.Cu at (314.8, 129.3)
- added R1: 1M, Resistor_SMD:R_0805_2012Metric, F.Cu at (294.4, 129.0)
- added R10: 130R, Resistor_SMD:R_0603_1608Metric, F.Cu at (284.8, 102.6)
- added R11: 5.1k, Resistor_SMD:R_0603_1608Metric, F.Cu at (288.8, 77.5)
- added R12: 130R, Resistor_SMD:R_0603_1608Metric, F.Cu at (288.8, 80.0)
- added R13: 02-LDR4, OptoDevice:R_LDR_5.1x4.3mm_P3.4mm_Vertical, F.Cu at (310.1, 115.2)
- added R14: 5.1k, Resistor_SMD:R_0603_1608Metric, F.Cu at (288.8, 82.5)
- added R15: 16k, Resistor_SMD:R_0603_1608Metric, F.Cu at (288.8, 85.1)
- added R15: 26.7k, Resistor_SMD:R_0603_1608Metric, F.Cu at (246.4, 148.2)
- added R16: 5.1k, Resistor_SMD:R_0603_1608Metric, F.Cu at (288.8, 87.6)
- added R16: 5.1k, Resistor_SMD:R_0603_1608Metric, F.Cu at (246.4, 146.6)
- added R17: 26.7k, Resistor_SMD:R_0603_1608Metric, F.Cu at (264.0, 148.2)
- added R18: 5.1k, Resistor_SMD:R_0603_1608Metric, F.Cu at (264.0, 146.6)
- added R19: 5.1k, Resistor_SMD:R_0603_1608Metric, F.Cu at (288.8, 95.1)
- added R2: 5.1k, Resistor_SMD:R_0603_1608Metric, F.Cu at (284.8, 82.5)
- added R20: 5.1k, Resistor_SMD:R_0603_1608Metric, F.Cu at (288.8, 97.6)
- added R21: 5.1k, Resistor_SMD:R_0603_1608Metric, F.Cu at (288.8, 100.1)
- added R22: 130R, Resistor_SMD:R_0603_1608Metric, F.Cu at (288.8, 102.6)
- added R23: 5.1k, Resistor_SMD:R_0603_1608Metric, F.Cu at (292.8, 77.5)
- added R24: 5.1k, Resistor_SMD:R_0603_1608Metric, F.Cu at (292.8, 80.0)
- added R25: 1k, Resistor_SMD:R_0603_1608Metric, F.Cu at (292.8, 82.5)
- added R26: 5.1k, Resistor_SMD:R_0603_1608Metric, F.Cu at (292.8, 85.1)
- added R27: 5.1k, Resistor_SMD:R_0603_1608Metric, F.Cu at (292.8, 87.6)
- added R28: 5.1k, Resistor_SMD:R_0603_1608Metric, F.Cu at (292.8, 90.1)
- added R29: 5.1k, Resistor_SMD:R_0603_1608Metric, F.Cu at (292.8, 92.6)
- added R3: 1k, Resistor_SMD:R_0603_1608Metric, F.Cu at (284.8, 85.1)
- added R4: 5.1k, Resistor_SMD:R_0603_1608Metric, F.Cu at (284.8, 87.6)
- added R5: 5.1k, Resistor_SMD:R_0603_1608Metric, F.Cu at (284.8, 90.1)
- added R6: 330R, Resistor_SMD:R_0603_1608Metric, F.Cu at (284.8, 92.6)
- added R7: 5.1k, Resistor_SMD:R_0603_1608Metric, F.Cu at (284.8, 95.1)
- added R8: 330R, Resistor_SMD:R_0603_1608Metric, F.Cu at (284.8, 97.6)
- added R9: 130R, Resistor_SMD:R_0603_1608Metric, F.Cu at (284.8, 100.1)
- added RV1: 10k, reck-switches:PT01-D130D-B103, F.Cu at (229.6, 108.7)
- added RV2: 10k, reck-switches:PT01-D130D-B103, F.Cu at (294.2, 110.2)
- added SW1: PTS810_SJM_250_SMTR_LFS, reck-switches:PTS810_SJM_250_SMTR_LFS, F.Cu at (312.1, 91.7)
- added SW2: PTS810_SJM_250_SMTR_LFS, reck-switches:PTS810_SJM_250_SMTR_LFS, F.Cu at (312.1, 96.4)
- added SW3: PTS810_SJM_250_SMTR_LFS, reck-switches:PTS810_SJM_250_SMTR_LFS, F.Cu at (312.1, 101.2)
- added TP1: TestPoint, TestPoint:TestPoint_Keystone_5000-5004_Miniature, F.Cu at (297.0, 78.4)
- added TP10: TestPoint, TestPoint:TestPoint_Keystone_5000-5004_Miniature, F.Cu at (310.1, 78.4)
- added TP11: TestPoint, TestPoint:TestPoint_Keystone_5000-5004_Miniature, F.Cu at (310.1, 82.8)
- added TP12: TestPoint, TestPoint:TestPoint_Keystone_5000-5004_Miniature, F.Cu at (310.1, 87.1)
- added TP13: TestPoint, TestPoint:TestPoint_Keystone_5000-5004_Miniature, F.Cu at (314.4, 78.4)
- added TP14: TestPoint, TestPoint:TestPoint_Keystone_5000-5004_Miniature, F.Cu at (314.4, 82.8)
- added TP15: TestPoint, TestPoint:TestPoint_Keystone_5000-5004_Miniature, F.Cu at (314.4, 87.1)
- added TP2: TestPoint, TestPoint:TestPoint_Keystone_5000-5004_Miniature, F.Cu at (297.0, 82.8)
- added TP3: TestPoint, TestPoint:TestPoint_Keystone_5000-5004_Miniature, F.Cu at (297.0, 87.1)
- added TP4: TestPoint, TestPoint:TestPoint_Keystone_5000-5004_Miniature, F.Cu at (301.4, 78.4)
- added TP5: TestPoint, TestPoint:TestPoint_Keystone_5000-5004_Miniature, F.Cu at (301.4, 82.8)
- added TP6: TestPoint, TestPoint:TestPoint_Keystone_5000-5004_Miniature, F.Cu at (301.4, 87.1)
- added TP7: TestPoint, TestPoint:TestPoint_Keystone_5000-5004_Miniature, F.Cu at (305.7, 78.4)
- added TP8: TestPoint, TestPoint:TestPoint_Keystone_5000-5004_Miniature, F.Cu at (305.7, 82.8)
- added TP9: TestPoint, TestPoint:TestPoint_Keystone_5000-5004_Miniature, F.Cu at (305.7, 87.1)
- added U1: USBLC6-2P6, Package_TO_SOT_SMD:SOT-666, F.Cu at (290.1, 129.3)
- added U10: WS2812B, reck-ics:WS2812B, F.Cu at (304.2, 119.2)
- added U11: DRV8231ADSGR, Package_SON:WSON-8-1EP_2x2mm_P0.5mm_EP0.9x1.6mm, F.Cu at (271.7, 129.1)
- added U12: WS2812B, reck-ics:WS2812B, F.Cu at (304.2, 125.3)
- added U13: VL53L0CXV0DH1, Sensor_Distance:ST_VL53L1x, F.Cu at (311.8, 120.2)
- added U14: MCP4725A0T-E/CH, Package_TO_SOT_SMD:SOT-23-6, F.Cu at (314.9, 124.7)
- added U15: ISM330DHCXTR, reck-ics:LGA-14_2.5x3.0mm_P0.5mm, F.Cu at (272.3, 120.8)
- added U16: BME280, Package_LGA:Bosch_LGA-8_2.5x2.5mm_P0.65mm_ClockwisePinNumbering, F.Cu at (271.8, 125.1)
- added U2: LCD2X16, reck-ics:LCD2X16, F.Cu at (266.0, 57.5)
- added U3: TPS62912RPUR, reck-ics:VQFN-HR-10_2x2mm, F.Cu at (250.0, 146.4)
- added U3: TPS62912RPUR, reck-ics:VQFN-HR-10_2x2mm, F.Cu at (310.6, 124.0)
- added U4: TPS62912RPUR, reck-ics:VQFN-HR-10_2x2mm, F.Cu at (267.6, 146.4)
- added U5: TXU0104PWR, Package_SO:TSSOP-14_4.4x5mm_P0.65mm, F.Cu at (240.1, 122.1)
- added U6: WS2812B, reck-ics:WS2812B, F.Cu at (304.2, 106.9)
- added U7: WS2812B, reck-ics:WS2812B, F.Cu at (304.2, 113.1)
- added U8: ESP32-S3-WROOM-2, RF_Module:ESP32-S3-WROOM-2, F.Cu at (250.0, 104.8)
- added U9: TXU0104PWR, Package_SO:TSSOP-14_4.4x5mm_P0.65mm, F.Cu at (240.1, 128.7)
Routing:
- net +5V-EXT: track 0.00 -> 39.0 mm, vias 0 -> 4
- net Net-(U4-FB): track 0.00 -> 6.94 mm
- net +12V-EXT: track 0.00 -> 5.20 mm
- net Net-(U4-NR/SS): track 0.00 -> 4.70 mm
- net GND: vias 0 -> 20
- added copper zone on F.Cu, net +12V-EXT
- added copper zone on F.Cu, net +5V-EXT
- added copper zone on F.Cu, net Net-(U4-SW)
Other:
- copper layers 2 -> 4
- rule pad_to_mask_clearance: 0 -> 0.05
