File: reck-pcba.kicad_sch (KiCad schematic)
At the start: 120 parts, among them J1 USB4105-GF-A, J2 575-4, J3 575-4, J4 Conn_01x03_Pin, J5 Conn_01x03_Pin, J6 TBL002A-350-02GR-2OR, Q1 BC846, SW1 PTS810_SJM_250_SMTR_LFS, SW2 PTS810_SJM_250_SMTR_LFS, SW3 PTS810_SJM_250_SMTR_LFS, U1 USBLC6-2P6, U10 WS2812B, U11 DRV8231ADSGR, U12 WS2812B, U13 VL53L0CXV0DH1, U14 MCP4725A0T-E/CH, U15 ISM330DHCXTR, U16 BME280, U2 LCD2X16, U3 TPS62912RPUR, U4 TPS62912RPUR, U5 TXU0104PWR, U6 WS2812B, U7 WS2812B, U8 ESP32-S3-WROOM-2, U9 TXU0104PWR

Commit message: updated
Parts:
- removed C10, C9: 1uF, symbol Device:C
- removed C13, C14, C16, C17, C18, C19: 22uF, symbol Device:C
- removed C2, C3, C4, C5: 10uF, symbol Device:C
- removed C7, C8: 2.2nF, symbol Device:C
- removed D8: D_Schottky, symbol Device:D_Schottky
- removed L1, L2: 2.2uH, symbol Device:L
- removed R13, R14: 6.04k, symbol Device:R
- removed R21: 16k, symbol Device:R
- removed R22, R24: 5.1k, symbol Device:R
- removed R23: 26.7k, symbol Device:R
- removed TP2: TestPoint, symbol Connector:TestPoint
- removed U3, U4: TPS62912RPUR, reck-ics:VQFN-HR-10_2x2mm, symbol reck-ics:TPS62912RPUR
- added D2, D9: CDBA340L-HF, Diode_SMD:D_SMA, symbol Device:D_Schottky
- added TP1, TP14, TP15: TestPoint, TestPoint:TestPoint_Keystone_5000-5004_Miniature, symbol Connector:TestPoint
- added U3: TPS564242DRLR, Package_TO_SOT_SMD:SOT-563, symbol reck-ics:TPS564242DRLR
- C1: value 4.7nF -> 2.2nF; footprint (none) -> Capacitor_SMD:C_0603_1608Metric
- C13: renamed from C11; footprint (none) -> Capacitor_SMD:C_0603_1608Metric
- C16: renamed from C12; footprint (none) -> Capacitor_SMD:C_0603_1608Metric
- C19: renamed from C15; footprint (none) -> Capacitor_SMD:C_0603_1608Metric
- C20, C21, C22, C23, C25, C27, C28, C29, C30, C31, C32, C33, C34, C35, C36, C6: footprint (none) -> Capacitor_SMD:C_0603_1608Metric
- C24, C37: footprint (none) -> Capacitor_SMD:C_0805_2012Metric
- C26: footprint (none) -> Capacitor_SMD:CP_Elec_6.3x5.9
- D1: footprint (none) -> LED_SMD:LED_0603_1608Metric
- D3: renamed from D2; footprint (none) -> LED_SMD:LED_0603_1608Metric
- D4: renamed from D3; value D_Schottky -> CDBA340L-HF; footprint (none) -> Diode_SMD:D_SMA
- D5: value D_Zener -> 1SMA5928BT3G; footprint (none) -> Diode_SMD:D_SMA
- D6: renamed from D4; footprint (none) -> LED_SMD:LED_0603_1608Metric
- D7: renamed from D6; footprint (none) -> LED_SMD:LED_0603_1608Metric
- D8: renamed from D7; footprint (none) -> LED_SMD:LED_0603_1608Metric
- R1: footprint (none) -> Resistor_SMD:R_0805_2012Metric
- R10, R12, R9: value 330R -> 130R; footprint (none) -> Resistor_SMD:R_0603_1608Metric
- R11, R2, R4, R5, R7: footprint (none) -> Resistor_SMD:R_0603_1608Metric
- R13: renamed from R15; footprint (none) -> OptoDevice:R_LDR_5.1x4.3mm_P3.4mm_Vertical
- R14: renamed from R16; footprint (none) -> Resistor_SMD:R_0603_1608Metric
- R19: renamed from R17; footprint (none) -> Resistor_SMD:R_0603_1608Metric
- R20: renamed from R18; footprint (none) -> Resistor_SMD:R_0603_1608Metric
- R21: renamed from R19; footprint (none) -> Resistor_SMD:R_0603_1608Metric
- R22: renamed from R20; value 330R -> 130R; footprint (none) -> Resistor_SMD:R_0603_1608Metric
- R23: renamed from R25; footprint (none) -> Resistor_SMD:R_0603_1608Metric
- R24: renamed from R26; footprint (none) -> Resistor_SMD:R_0603_1608Metric
- R25: renamed from R27; footprint (none) -> Resistor_SMD:R_0603_1608Metric
- R26: renamed from R28; footprint (none) -> Resistor_SMD:R_0603_1608Metric
- R27: renamed from R29; footprint (none) -> Resistor_SMD:R_0603_1608Metric
- R28: renamed from R30; footprint (none) -> Resistor_SMD:R_0603_1608Metric
- R29: renamed from R31; footprint (none) -> Resistor_SMD:R_0603_1608Metric
- R3: value 3.3k -> 1k; footprint (none) -> Resistor_SMD:R_0603_1608Metric
- R6, R8: value 1k -> 330R; footprint (none) -> Resistor_SMD:R_0603_1608Metric
- RV1, RV2: footprint (none) -> reck-switches:PT01-D130D-B103
- TP10, TP11, TP12, TP13, TP3, TP4, TP5, TP6, TP7, TP8, TP9: footprint (none) -> TestPoint:TestPoint_Keystone_5000-5004_Miniature
- TP2: renamed from TP1; footprint (none) -> TestPoint:TestPoint_Keystone_5000-5004_Miniature
- U15: footprint reck-ics:LGA-14L_2.5x3.0mm_P0.5mm -> reck-ics:LGA-14_2.5x3.0mm_P0.5mm
Connections:
- net +3V3: now also D9.1 (K)
- net +VBUS: now also D2.1 (K); no longer J1.A4 (VBUS), J1.A9 (VBUS), J1.B4 (VBUS), J1.B9 (VBUS)
- net GND: now also TP14.1, TP15.1; no longer TP12.1
- net MOTOR-IN2: now also TP3.1
- net PWM-BUZZER: no longer TP3.1
- net PWM-SERVO: now also TP12.1
- net PWM-SERVO-5V: now also TP13.1
- net V-DAC: now also TP1.1; no longer TP13.1
- net at BZ1.2, Q1.3 (C): now also D9.2 (A)
- new net +VBUS-CONN: D2.2 (A), J1.A4 (VBUS), J1.A9 (VBUS), J1.B4 (VBUS), J1.B9 (VBUS)
- no-connect marks 19 -> 17
Other:
- note removed: "Buck Regulators"
- note removed: "I2C Pullups"
- note removed: "MISO Pullup"
- note removed: "Step-down Power Conversion"
- moved on the sheet: BZ1, D4, D5, J2, J3, TP2
